Commit message: ~6.3.2

File: learning/6_sim/src/description/urdf/bot/base.urdf.xacro (robot description, xacro)
@@ -2,4 +2,6 @@
 <robot xmlns:xacro="http://www.ros.org/wiki/xacro">
     <xacro:macro name="base_xacro" params="length radius">
+        <!-- 虚拟 -->
+        <link name="base_foot_print"/>
         <link name="base_link">
             <visual>
@@ -12,5 +14,22 @@
                 </material>
             </visual>
+            <!-- 碰撞 -->
+            <collision>
+                <origin rpy="0 0 0" xyz="0 0 0"/>
+                <geometry>
+                    <cylinder radius="${radius}" length="${length}"/>
+                </geometry>
+                <material name="white">
+                    <color rgba="1.0 1.0 1.0 0.5"/>
+                </material>
+            </collision>
+            <!-- 质量(惯性) -->
+            <xacro:cylinder_inertia m="1.0" r="${radius}" l="${length}"/>
         </link>
+        <joint name="base_print_joint" type="fixed">
+            <parent link="base_foot_print"/>
+            <child link="base_link"/>
+            <origin rpy="0 0 0" xyz="0 0 ${length/2+0.032-0.01}"/>
+        </joint>
     </xacro:macro>
 </robot>

File: learning/6_sim/src/description/urdf/bot/bot.urdf.xacro (robot description, xacro)
@@ -7,4 +7,5 @@
 <xacro:include filename="$(find description)/urdf/bot/actuators/wheel.urdf.xacro"/>
 <xacro:include filename="$(find description)/urdf/bot/actuators/caster.urdf.xacro"/>
+<xacro:include filename="$(find description)/urdf/common_inertial.urdf.xacro"/>
 <xacro:base_xacro length="0.12" radius="0.10"/>
 <xacro:lidar_xacro xyz="0 0 0.1" />
