Commit message: gazebo版本不同，调整plugin

File: learning/6_sim/src/description/urdf/bot/actuators/wheel.urdf.xacro (robot description, xacro)
@@ -19,4 +19,14 @@
             <axis xyz="0 1 0"/>
         </joint>
+        <gazebo reference="${wheel_name}_link">
+            <material>Gazebo/green</material>
+            <!-- 摩擦系数（1：切向；2：法向） -->
+            <mu1 value="20"/>
+            <mu2 value="20"/>
+            <!-- 刚度 -->
+            <kp value="1000000000"/>
+            <!-- 阻尼 -->
+            <kd value="20"/>
+        </gazebo>
     </xacro:macro>
 </robot>

File: learning/6_sim/src/description/urdf/bot/base.urdf.xacro (robot description, xacro)
@@ -25,5 +25,5 @@
             </collision>
             <!-- 质量(惯性) -->
-            <xacro:cylinder_inertia m="1.0" r="${radius}" l="${length}"/>
+            <xacro:cylinder_inertia m="1.0" r="${radius}" h="${length}"/>
         </link>
         <joint name="base_print_joint" type="fixed">

File: learning/6_sim/src/description/urdf/bot/bot.urdf.xacro (robot description, xacro)
@@ -7,5 +7,7 @@
 <xacro:include filename="$(find description)/urdf/bot/actuators/wheel.urdf.xacro"/>
 <xacro:include filename="$(find description)/urdf/bot/actuators/caster.urdf.xacro"/>
-<xacro:include filename="$(find description)/urdf/common_inertial.urdf.xacro"/>
+<xacro:include filename="$(find description)/urdf/bot/plugin/common_inertial.urdf.xacro"/>
+<xacro:include filename="$(find description)/urdf/bot/plugin/gz_control_plugin.xacro"/>
+<xacro:include filename="$(find description)/urdf/bot/plugin/gz_sensors_plugin.xacro"/>
 <xacro:base_xacro length="0.12" radius="0.10"/>
 <xacro:lidar_xacro xyz="0 0 0.1" />
@@ -16,3 +18,5 @@
 <xacro:caster_xacro caster_name="caster_front" xyz="-0.08 0 0.76" />
 <xacro:caster_xacro caster_name="caster_right" xyz="-0.08 -0.1 0.76" />
+<xacro:gazebo_control_plugin/>
+<xacro:gazebo_sensor_plugin/>
 </robot>

File: learning/6_sim/src/description/urdf/bot/sensors/laser.urdf.xacro (robot description, xacro)
@@ -39,4 +39,10 @@
             <origin rpy="0 0 0" xyz="${xyz}"/>
         </joint>
+        <gazebo reference="lidar_bear_link">
+            <material>Gazebo/Black</material>
+        </gazebo>
+        <gazebo reference="lidar_link">
+            <material>Gazebo/Black</material>
+        </gazebo>
     </xacro:macro>
 </robot>
